Commit message: ffe

File: arm_and_gripper/arm_and_gripper/urdf/robotiq_85_gripper/robotiq_85_gripper.urdf.xacro (robot description, xacro)
@@ -47,4 +47,5 @@
         <geometry>
           <mesh filename="package://arm_and_gripper/meshes/robotiq_85_gripper/visual/robotiq_85_knuckle_link.dae"/>
+          <!-- <mesh filename="$(find arm_and_gripper)/meshes/robotiq_85_gripper/visual/robotiq_85_knuckle_link.dae"/> -->
         </geometry>
       </visual>
@@ -52,4 +53,5 @@
         <geometry>
           <mesh filename="package://arm_and_gripper/meshes/robotiq_85_gripper/collision/robotiq_85_knuckle_link.stl"/>
+          <!-- <mesh filename="$(find arm_and_gripper)/meshes/robotiq_85_gripper/visual/robotiq_85_knuckle_link.dae"/> -->
         </geometry>
       </collision>

File: arm_and_gripper/arm_and_gripper/urdf/ur3e.urdf.xacro (robot description, xacro)
@@ -56,4 +56,5 @@
         <geometry>
           <mesh filename="package://arm_and_gripper/meshes/ur3e/visual/base.dae"/>
+          <!-- <mesh filename="$(find arm_and_gripper)/meshes/ur3e/visual/base.dae"/> -->
         </geometry>
         <material name="LightGrey">
@@ -65,4 +66,5 @@
         <geometry>
           <mesh filename="package://arm_and_gripper/meshes/ur3e/visual/base.dae"/>
+          <!-- <mesh filename="$(find arm_and_gripper)/meshes/ur3e/visual/base.dae"/> -->
         </geometry>
       </collision>
